Commit message: Laser output in youbot namespace - issue #1

File: youbot_description/gazebo/gazebo.urdf.xacro (robot description, xacro)
@@ -1,15 +1,8 @@
 <?xml version="1.0"?>
-<robot xmlns:xacro="http://ros.org/wiki/xacro">
-  <gazebo>
-    <plugin name="gazebo_ros_controller_manager" filename="libgazebo_ros_control.so">
-      <robotNamespace>/youbot</robotNamespace>
-    </plugin>
-    <plugin name="object_controller" filename="libgazebo_ros_planar_move.so">
-      <commandTopic>cmd_vel</commandTopic>
-      <odometryTopic>odom</odometryTopic>
-      <odometryFrame>odom</odometryFrame>
-      <odometryRate>20.0</odometryRate>
-      <robotBaseFrame>base_footprint</robotBaseFrame>
-    </plugin>
-  </gazebo>
+<robot name="youbot" xmlns:xacro="http://ros.org/wiki/xacro">
+    <gazebo>
+        <plugin name="gazebo_ros_controller_manager" filename="libgazebo_ros_control.so">
+            <robotNamespace>/youbot</robotNamespace>
+        </plugin>
+    </gazebo>
 </robot>

File: youbot_description/urdf/sensors/hokuyo_urg04_laser.gazebo.xacro (robot description, xacro)
@@ -4,32 +4,33 @@
        xmlns:interface="http://playerstage.sourceforge.net/gazebo/xmlschema/#interface"
        xmlns:xacro="http://ros.org/wiki/xacro">
-  <xacro:macro name="hokuyo_urg04_laser_gazebo" params="name ros_topic update_rate min_angle max_angle">
-    <gazebo reference="${name}_link">
-      <sensor name="${name}" type="ray">
-	<ray>
-	  <scan>
-	    <horizontal>
-		<samples>640</samples>
-		<resolution>1.0</resolution>
-		<min_angle>${min_angle*180.0/M_PI}</min_angle>
-		<max_angle>${max_angle*180.0/M_PI}</max_angle>
-	    </horizontal>
-	  </scan>
-	  <range>
-		<min>0.05</min>
-		<max>5.6</max>
-		<resolution>0.36</resolution>
-	  </range>
-	</ray>
-	<plugin name="gazebo_ros_${name}_controller" filename="libgazebo_ros_laser.so">
-	  <gaussianNoise>0.000</gaussianNoise>
-	  <alwaysOn>true</alwaysOn>
-	  <updateRate>${update_rate}</updateRate>
-	  <topicName>${ros_topic}</topicName>
-	  <frameName>/${name}_link</frameName>
-	  <interface:laser name="gazebo_ros_${name}_iface" />
-        </plugin>
-      </sensor>
-    </gazebo>
-  </xacro:macro>
+    <xacro:macro name="hokuyo_urg04_laser_gazebo" params="name ros_topic update_rate min_angle max_angle">
+        <gazebo reference="${name}_link">
+            <sensor name="${name}" type="ray">
+                <ray>
+                    <scan>
+                        <horizontal>
+                            <samples>640</samples>
+                            <resolution>1.0</resolution>
+                            <min_angle>${min_angle*180.0/M_PI}</min_angle>
+                            <max_angle>${max_angle*180.0/M_PI}</max_angle>
+                        </horizontal>
+                    </scan>
+                    <range>
+                        <min>0.05</min>
+                        <max>5.6</max>
+                        <resolution>0.36</resolution>
+                    </range>
+                </ray>
+                <plugin name="gazebo_ros_${name}_controller" filename="libgazebo_ros_laser.so">
+                    <robotNamespace>/youbot</robotNamespace>
+                    <gaussianNoise>0.000</gaussianNoise>
+                    <alwaysOn>true</alwaysOn>
+                    <updateRate>${update_rate}</updateRate>
+                    <topicName>${ros_topic}</topicName>
+                    <frameName>/${name}_link</frameName>
+                    <interface:laser name="gazebo_ros_${name}_iface" />
+                </plugin>
+            </sensor>
+        </gazebo>
+    </xacro:macro>
 </robot>

File: youbot_description/urdf/sensors/hokuyo_urg04_laser.urdf.xacro (robot description, xacro)
@@ -1,7 +1,4 @@
 <?xml version="1.0"?>
-<robot xmlns:sensor="http://playerstage.sourceforge.net/gazebo/xmlschema/#sensor"
-       xmlns:controller="http://playerstage.sourceforge.net/gazebo/xmlschema/#controller"
-       xmlns:interface="http://playerstage.sourceforge.net/gazebo/xmlschema/#interface"
-       xmlns:xacro="http://ros.org/wiki/xacro">
+<robot name="youbot" xmlns:xacro="http://ros.org/wiki/xacro">
   <include filename="$(find youbot_description)/urdf/sensors/hokuyo_urg04_laser.gazebo.xacro" />
   <xacro:macro name="hokuyo_urg04_laser" params="name parent *origin ros_topic update_rate min_angle max_angle">

File: youbot_description/urdf/youbot_base/base.urdf.xacro (robot description, xacro)
@@ -228,6 +228,4 @@
       </inertial>
     </link>
-    <gazebo reference = "caster_link_br">
-    </gazebo>
     <joint name="wheel_joint_br" type="continuous">
       <axis xyz="0 1 0" />
@@ -258,6 +256,4 @@
       </collision>
     </link>
-    <gazebo reference = "wheel_link_br">
-    </gazebo>
     <!-- base laser front -->
     <xacro:hokuyo_urg04_laser name="${name}_laser_front" parent="${name}" ros_topic="scan_front" update_rate="10" min_angle="-1.57" max_angle="1.57" >
