Commit message: set gravity and selfcollision to true in most of the model links
These changes only affect Gazebo as these are properties of the
<gazebo> tag. selfcollision should avoid the robot collapsing into
itself.

File: youbot_description/urdf/youbot_arm/arm.gazebo.xacro (robot description, xacro)
@@ -2,23 +2,27 @@
 <robot name="youbot" xmlns:xacro="http://ros.org/wiki/xacro">
 	<xacro:macro name="youbot_arm_gazebo" params="name">
-		<gazebo>
-			<link name="${name}_link_0">
-				<gravity>false</gravity>
-			</link>
+		<gazebo reference="${name}_link_0">
+			<gravity>true</gravity>
+			<selfCollide>true</selfCollide>
 		</gazebo>
 		<gazebo reference="${name}_link_1">
-			<gravity>false</gravity>
+			<gravity>true</gravity>
+			<selfCollide>true</selfCollide>
 		</gazebo>
 		<gazebo reference="${name}_link_2">
-			<gravity>false</gravity>
+			<gravity>true</gravity>
+			<selfCollide>true</selfCollide>
 		</gazebo>
 		<gazebo reference="${name}_link_3">
-			<gravity>false</gravity>
+			<gravity>true</gravity>
+			<selfCollide>true</selfCollide>
 		</gazebo>
 		<gazebo reference="${name}_link_4">
-			<gravity>false</gravity>
+			<gravity>true</gravity>
+			<selfCollide>true</selfCollide>
 		</gazebo>
 		<gazebo reference="${name}_link_5">
-			<gravity>false</gravity>
+			<gravity>true</gravity>
+			<selfCollide>true</selfCollide>
 		</gazebo>
 	</xacro:macro>

File: youbot_description/urdf/youbot_base/base.gazebo.xacro (robot description, xacro)
@@ -11,4 +11,8 @@
         <robotBaseFrame>base_footprint</robotBaseFrame>
       </plugin>
+    </gazebo>
+    <gazebo reference="${name}_footprint">
+      <gravity>true</gravity>
+      <selfCollide>true</selfCollide>
     </gazebo>
     <!-- old position controller -->

File: youbot_description/urdf/youbot_gripper/gripper.gazebo.xacro (robot description, xacro)
@@ -1,21 +1,18 @@
 <?xml version="1.0"?>
-<robot xmlns:sensor="http://playerstage.sourceforge.net/gazebo/xmlschema/#sensor"
-       xmlns:controller="http://playerstage.sourceforge.net/gazebo/xmlschema/#controller"
-       xmlns:interface="http://playerstage.sourceforge.net/gazebo/xmlschema/#interface"
-       xmlns:xacro="http://ros.org/wiki/xacro">
+<robot name="youbot" xmlns:xacro="http://ros.org/wiki/xacro">
 	<xacro:macro name="youbot_gripper_gazebo" params="name">
 		<gazebo reference="${name}_palm_link">
 			<material>Gazebo/Black</material>
-			<gravity>false</gravity>
+			<gravity>true</gravity>
 			<selfCollide>true</selfCollide>
 		</gazebo>
 		<gazebo reference="${name}_finger_l_link">
 			<material>Gazebo/Black</material>
-			<gravity>false</gravity>
+			<gravity>true</gravity>
 			<selfCollide>true</selfCollide>
 		</gazebo>
 		<gazebo reference="${name}_finger_r_link">
 			<material>Gazebo/Black</material>
-			<gravity>false</gravity>
+			<gravity>true</gravity>
 			<selfCollide>true</selfCollide>
 		</gazebo>

File: youbot_description/urdf/youbot_gripper/gripper.urdf.xacro (robot description, xacro)
@@ -1,7 +1,4 @@
 <?xml version="1.0"?>
-<robot xmlns:sensor="http://playerstage.sourceforge.net/gazebo/xmlschema/#sensor"
-	xmlns:controller="http://playerstage.sourceforge.net/gazebo/xmlschema/#controller"
-	xmlns:interface="http://playerstage.sourceforge.net/gazebo/xmlschema/#interface"
-	xmlns:xacro="http://ros.org/wiki/xacro">
+<robot name="youbot" xmlns:xacro="http://ros.org/wiki/xacro">
 	<include filename="$(find youbot_description)/urdf/youbot_gripper/gripper.gazebo.xacro" />
 	<include filename="$(find youbot_description)/urdf/youbot_gripper/gripper.transmission.xacro" />
@@ -35,6 +32,4 @@
 			</collision>
 		</link>
-		<gazebo reference = "${name}_palm_link">
-		</gazebo>
 <!--
 		<link name="${name}_camera_collision_box_link">
@@ -84,6 +79,4 @@
 		</collision>
 	</link>
-	<gazebo reference = "${name}_finger_link_l">
-	</gazebo>
 	<joint name="${name}_finger_joint_r" type="prismatic">
 		<origin xyz="0.046 -0.010 0.003" rpy="0 ${M_PI / 2} 0" />
@@ -115,6 +108,4 @@
 		</collision>
 	</link>
-	<gazebo reference = "${name}_finger_link_r">
-	</gazebo>
 	<!-- asus xtion camera
 	<xacro:asus_xtion_camera name="xtion" parent="${name}_palm_link" tilt="0.0">

File: youbot_description/urdf/youbot_plate/plate.urdf.xacro (robot description, xacro)
@@ -1,4 +1,5 @@
 <?xml version="1.0"?>
 <robot name="youbot" xmlns:xacro="http://www.ros.org/wiki/xacro">
+	<include filename="$(find youbot_description)/urdf/youbot_plate/plate.gazebo.xacro" />
 	<xacro:macro name="youbot_plate" params="parent name *origin">
 		<!-- joint between arm_7_link and sdh_palm_link -->
@@ -27,4 +28,5 @@
 			</collision>
 		</link>
+		<xacro:youbot_plate_gazebo name="${name}" />
 	</xacro:macro>
 </robot>
