Commit message: removed limit on effort for arm joints
Removing limits on efforts, while leaving the ones on velocity there
solve the issue with slow joints. If this brings other problems, the
only solution is go back to normal limits and check for weights and
inertia matrices.

File: youbot_description/urdf/youbot_arm/arm.urdf.xacro (robot description, xacro)
@@ -43,5 +43,5 @@
 			<!-- damping - N*s/m, N*s*m/rad -->
 			<!-- friction - N, N*m -->
-			<limit effort="${9.5}" velocity="${M_PI / 2.0}" lower="0" upper="${joint_1_limit}"/>
+			<limit effort="${10000}" velocity="${M_PI / 2.0}" lower="0" upper="${joint_1_limit}"/>
 			<!--effort - N, N*m-->
 			<!--velocity - m/s, rad/s-->
@@ -79,5 +79,5 @@
 			<!--<calibration rising="${arm_2_ref}" falling="${arm_2_ref}"/>-->
 			<dynamics damping="1" friction="1" />
-			<limit effort="${9.5}" velocity="${M_PI / 2.0}" lower="0" upper="${joint_2_limit}"/>
+			<limit effort="${10000}" velocity="${M_PI / 2.0}" lower="0" upper="${joint_2_limit}"/>
 			<safety_controller k_position="20" k_velocity="${2*9.5/M_PI}" soft_lower_limit="${threshold}" soft_upper_limit="${joint_2_limit_soft}" />
 		</joint>
@@ -108,5 +108,5 @@
 			<axis xyz="0 1 0"/>
 			<dynamics damping="1" friction="1" />
-			<limit effort="${6}" velocity="${M_PI / 2.0}" lower="-${joint_3_limit}" upper="0"/>
+			<limit effort="${10000}" velocity="${M_PI / 2.0}" lower="-${joint_3_limit}" upper="0"/>
 			<safety_controller k_position="20" k_velocity="50" soft_lower_limit="-${joint_3_limit_soft}" soft_upper_limit="-${threshold}" />
 		</joint>
@@ -139,5 +139,5 @@
 			<!--<calibration rising="${arm_4_ref}" falling="${arm_4_ref}"/>-->
 			<dynamics damping="1" friction="1" />
-			<limit effort="${2}" velocity="${M_PI / 2.0}" lower="0" upper="${joint_4_limit}"/>
+			<limit effort="${10000}" velocity="${M_PI / 2.0}" lower="0" upper="${joint_4_limit}"/>
 			<safety_controller k_position="20" k_velocity="100" soft_lower_limit="0" soft_upper_limit="${joint_4_limit_soft}" />
 		</joint>
@@ -170,5 +170,5 @@
 			<!--<calibration rising="${arm_5_ref}" falling="${arm_5_ref}"/>-->
 			<dynamics damping="1" friction="1" />
-			<limit effort="1" velocity="${M_PI / 2.0}" lower="0" upper="${joint_5_limit}" />
+			<limit effort="${10000}" velocity="${M_PI / 2.0}" lower="0" upper="${joint_5_limit}" />
 			<safety_controller k_position="20" k_velocity="100" soft_lower_limit="0" soft_upper_limit="${joint_5_limit_soft}" />
 		</joint>
