Commit message: fixed caster joints for mecanum wheels
As mecanum wheels don't use caster joints, I fixed the caster joints in the model and removed the relative transmissions. Close issue #9

File: youbot_description/urdf/youbot_base/base.transmission.xacro (robot description, xacro)
@@ -14,12 +14,4 @@
       </actuator>
     </transmission>
-    <transmission name="caster_trans_fl">
-      <type>transmission_interface/SimpleTransmission</type>
-      <joint name="caster_joint_fl"/>
-      <actuator name="caster_motor_fl">
-        <hardwareInterface>EffortJointInterface</hardwareInterface>
-        <mechanicalReduction>${caster_mechanical_reduction}</mechanicalReduction>
-      </actuator>
-    </transmission>
     <!-- front right wheel -->
     <transmission name="wheel_trans_fr">
@@ -29,12 +21,4 @@
         <hardwareInterface>EffortJointInterface</hardwareInterface>
         <mechanicalReduction>${wheel_mechanical_reduction}</mechanicalReduction>
-      </actuator>
-    </transmission>
-    <transmission name="caster_trans_fr">
-      <type>transmission_interface/SimpleTransmission</type>
-      <joint name="caster_joint_fr"/>
-      <actuator name="caster_motor_fr">
-        <hardwareInterface>EffortJointInterface</hardwareInterface>
-        <mechanicalReduction>${caster_mechanical_reduction}</mechanicalReduction>
       </actuator>
     </transmission>
@@ -48,12 +32,4 @@
       </actuator>
     </transmission>
-    <transmission name="caster_trans_bl">
-      <type>transmission_interface/SimpleTransmission</type>
-      <joint name="caster_joint_bl"/>
-      <actuator name="caster_motor_bl">
-        <hardwareInterface>EffortJointInterface</hardwareInterface>
-        <mechanicalReduction>${caster_mechanical_reduction}</mechanicalReduction>
-      </actuator>
-    </transmission>
     <!-- back right wheel -->
     <transmission name="wheel_trans_br">
@@ -65,12 +41,4 @@
       </actuator>
     </transmission>
-    <transmission name="caster_trans_br">
-      <type>transmission_interface/SimpleTransmission</type>
-      <joint name="caster_joint_br"/>
-      <actuator name="caster_motor_br">
-        <hardwareInterface>EffortJointInterface</hardwareInterface>
-        <mechanicalReduction>${caster_mechanical_reduction}</mechanicalReduction>
-      </actuator>
-    </transmission>
   </xacro:macro>
 </robot>

File: youbot_description/urdf/youbot_base/base.urdf.xacro (robot description, xacro)
@@ -76,10 +76,7 @@
     </link>
     <!-- front left wheel -->
-    <joint name="caster_joint_fl" type="continuous">
+    <joint name="caster_joint_fl" type="fixed">
       <origin xyz="${caster_offset_x} ${caster_offset_y} ${caster_offset_z}" rpy="0 0 0" />
       <axis xyz="0 0 1" />
-      <limit effort="${caster_joint_effort}" velocity="${caster_joint_velocity}"/>
-      <dynamics damping="${caster_joint_damping}" friction="${caster_joint_friction}" />
-      <safety_controller k_velocity="${caster_joint_safety_k_velocity}" />
       <parent link="${name}_link"/>
       <child link="caster_link_fl" />
@@ -121,10 +118,7 @@
     </link>
     <!-- front right wheel -->
-    <joint name="caster_joint_fr" type="continuous">
+    <joint name="caster_joint_fr" type="fixed">
       <origin xyz="${caster_offset_x} ${-caster_offset_y} ${caster_offset_z}" rpy="0 0 0" />
       <axis xyz="0 0 1" />
-      <limit effort="${caster_joint_effort}" velocity="${caster_joint_velocity}"/>
-      <dynamics damping="${caster_joint_damping}" friction="${caster_joint_friction}" />
-      <safety_controller k_velocity="${caster_joint_safety_k_velocity}" />
       <parent link="${name}_link"/>
       <child link="caster_link_fr" />
@@ -166,10 +160,7 @@
     </link>
     <!-- back left wheel -->
-    <joint name="caster_joint_bl" type="continuous">
+    <joint name="caster_joint_bl" type="fixed">
       <origin xyz="${-caster_offset_x} ${caster_offset_y} ${caster_offset_z}" rpy="0 0 0" />
       <axis xyz="0 0 1" />
-      <limit effort="${caster_joint_effort}" velocity="${caster_joint_velocity}"/>
-      <dynamics damping="${caster_joint_damping}" friction="${caster_joint_friction}" />
-      <safety_controller k_velocity="${caster_joint_safety_k_velocity}" />
       <parent link="${name}_link"/>
       <child link="caster_link_bl" />
@@ -212,10 +203,7 @@
     </link>
     <!-- back right wheel -->
-    <joint name="caster_joint_br" type="continuous">
+    <joint name="caster_joint_br" type="fixed">
       <origin xyz="${-caster_offset_x} ${-caster_offset_y} ${caster_offset_z}" rpy="0 0 0" />
       <axis xyz="0 0 1" />
-      <limit effort="${caster_joint_effort}" velocity="${caster_joint_velocity}"/>
-      <dynamics damping="${caster_joint_damping}" friction="${caster_joint_friction}" />
-      <safety_controller k_velocity="${caster_joint_safety_k_velocity}" />
       <parent link="${name}_link"/>
       <child link="caster_link_br" />
