Commit message: plate and youbot launch

File: youbot_description/robots/youbot.urdf.xacro (robot description, xacro)
@@ -1,6 +1,6 @@
 <?xml version="1.0"?>
+<!-- Refactored by Arn-O -->
 <robot name="youbot" xmlns:xacro="http://www.ros.org/wiki/xacro">
   <!-- The following included files set up definitions of parts of the robot body -->
-  <!-- misc common stuff? -->
   <xacro:include filename="$(find youbot_description)/urdf/common.xacro" />
   <!-- youbot base -->
@@ -8,28 +8,7 @@
   <!-- youbot plate -->
   <xacro:include filename="$(find youbot_description)/urdf/youbot_plate/plate.urdf.xacro" />
-  <!-- youbot arm -->
-  <xacro:include filename="$(find youbot_description)/urdf/youbot_arm/arm.urdf.xacro"/>
-  <!-- youbot gripper -->
-  <xacro:include filename="$(find youbot_description)/urdf/youbot_gripper/gripper.urdf.xacro" />
   <!-- generic simulator_gazebo plugins for starting mechanism control, ros time, ros battery -->
   <xacro:include filename="$(find youbot_description)/gazebo/gazebo.urdf.xacro" />
-  <!-- Now we can start using the macros included above to define the actual youbot -->
-  <!-- The first use of a macro.  This one was defined in base.urdf.xacro above.
-       A macro like this will expand to a set of link and joint definitions, and to additional
-       Gazebo-related extensions (sensor plugins, etc).  The macro takes an argument, name,
-       that equals "base", and uses it to generate names for its component links and joints
-       (e.g., base_link).  The included origin block is also an argument to the macro.  By convention,
-       the origin block defines where the component is w.r.t its parent (in this case the parent
-       is the world frame). For more, see http://www.ros.org/wiki/xacro -->
-<!-- foot for arm-->
-  <xacro:youbot_base name="base"/>
-  <xacro:youbot_plate name="plate" parent="base_link">
-    <origin xyz="-0.159 0 0.055" rpy="0 0 0" />
-  </xacro:youbot_plate>
-  <xacro:youbot_arm name="arm" parent="base_link">
-     <origin xyz="0.143 0 0.046" rpy="0 0 0" />
-  </xacro:youbot_arm>
-  <xacro:youbot_gripper name="gripper" parent="arm_link_5">
-    <origin xyz="-0.0027 0 .016" rpy="0 ${-M_PI/2} ${M_PI}" />
-  </xacro:youbot_gripper>
+  <xacro:youbot_base />
+  <xacro:youbot_plate />
 </robot>

File: youbot_description/urdf/youbot_base/base.gazebo.xacro (robot description, xacro)
@@ -9,5 +9,5 @@
         <odometryFrame>odom</odometryFrame>
         <odometryRate>20.0</odometryRate>
-        <robotBaseFrame>base_link</robotBaseFrame>
+        <robotBaseFrame>base_footprint</robotBaseFrame>
       </plugin>
     </gazebo>

File: youbot_description/urdf/youbot_base/base.urdf.xacro (robot description, xacro)
@@ -3,17 +3,26 @@
 <robot name="youbot" xmlns:xacro="http://www.ros.org/wiki/xacro">
   <!-- includes -->
-  <xacro:include filename="$(find youbot_description)/urdf/youbot_base/specs.urdf.xacro" />
+  <xacro:include filename="$(find youbot_description)/urdf/specs.urdf.xacro" />
   <xacro:include filename="$(find youbot_description)/urdf/youbot_base/base.gazebo.xacro" />
   <xacro:macro name="youbot_base">
     <!-- ### links ### -->
     <!-- base -->
-    <link name="base_link">
+    <link name="base_footprint">
+      <inertial>
+        <mass value="0.001" />
+        <inertia ixx="0.010" ixy="0.000" ixz="0.000" iyy="0.010" iyz="0.000" izz="0.010" />
+      </inertial>
+      <visual>
+        <geometry>
+          <box size="0.001 0.001 0.001" />
+        </geometry>
+      </visual>
+    </link>
+   <link name="base_link">
       <inertial>
         <mass value="${base_mass}" />
-        <origin xyz="${base_pose_x} ${base_pose_y} ${base_pose_z}" />
         <inertia ixx="1.000" ixy="0.000" ixz="0.000" iyy="1.000" iyz="0.000" izz="1.000" />
       </inertial>
       <visual>
-        <origin xyz="0 0 0" rpy="0 0 0" />
         <geometry>
           <mesh filename="package://youbot_description/meshes/youbot_base/base_frame.dae"/>
@@ -39,5 +48,61 @@
       </collision>
     </link>
+    <!-- front right wheel -->
+    <link name="wheel_link_fr">
+      <inertial>
+        <mass value="${wheel_mass}" />
+        <inertia  ixx="0.010" ixy="0.000" ixz="0.000" iyy="0.010" iyz="0.000" izz="0.010" />
+      </inertial>
+      <visual>
+        <geometry>
+          <sphere radius="${wheel_radius}" />
+        </geometry>
+      </visual>
+      <collision>
+        <geometry>
+          <sphere radius="${wheel_radius}" />
+        </geometry>
+      </collision>
+    </link>
+    <!-- back left wheel -->
+    <link name="wheel_link_bl">
+      <inertial>
+        <mass value="${wheel_mass}" />
+        <inertia  ixx="0.010" ixy="0.000" ixz="0.000" iyy="0.010" iyz="0.000" izz="0.010" />
+      </inertial>
+      <visual>
+        <geometry>
+          <sphere radius="${wheel_radius}" />
+        </geometry>
+      </visual>
+      <collision>
+        <geometry>
+          <sphere radius="${wheel_radius}" />
+        </geometry>
+      </collision>
+    </link>
+    <!-- back right wheel -->
+    <link name="wheel_link_br">
+      <inertial>
+        <mass value="${wheel_mass}" />
+        <inertia  ixx="0.010" ixy="0.000" ixz="0.000" iyy="0.010" iyz="0.000" izz="0.010" />
+      </inertial>
+      <visual>
+        <geometry>
+          <sphere radius="${wheel_radius}" />
+        </geometry>
+      </visual>
+      <collision>
+        <geometry>
+          <sphere radius="${wheel_radius}" />
+        </geometry>
+      </collision>
+    </link>
     <!-- ### joints ### -->
+    <joint name="base_joint" type="fixed">
+      <origin xyz="${base_pose_x} ${base_pose_y} ${base_pose_z}" rpy="0 0 0" />
+      <parent link="base_footprint"/>
+      <child link="base_link" />
+    </joint>
     <joint name="wheel_fl_joint" type="fixed">
       <origin xyz="${wheel_fl_pose_x} ${wheel_fl_pose_y} ${wheel_fl_pose_z}" rpy="0 0 0" />
@@ -45,126 +110,21 @@
       <child link="wheel_link_fl" />
     </joint>
+    <joint name="wheel_fr_joint" type="fixed">
+      <origin xyz="${wheel_fr_pose_x} ${wheel_fr_pose_y} ${wheel_fr_pose_z}" rpy="0 0 0" />
+      <parent link="base_link"/>
+      <child link="wheel_link_fr" />
+    </joint>
+    <joint name="wheel_bl_joint" type="fixed">
+      <origin xyz="${wheel_bl_pose_x} ${wheel_bl_pose_y} ${wheel_bl_pose_z}" rpy="0 0 0" />
+      <parent link="base_link"/>
+      <child link="wheel_link_bl" />
+    </joint>
+    <joint name="wheel_br_joint" type="fixed">
+      <origin xyz="${wheel_br_pose_x} ${wheel_br_pose_y} ${wheel_br_pose_z}" rpy="0 0 0" />
+      <parent link="base_link"/>
+      <child link="wheel_link_br" />
+    </joint>
+    <!-- extensions -->
     <xacro:youbot_base_gazebo />
   </xacro:macro>
 </robot>
-<!--
-    <link name="${name}_footprint">
-      <inertial>
-        <mass value="0.0001" />
-        <origin xyz="0 0 ${-base_size_z / 2.0}" rpy="0 0 0" />
-        <inertia ixx="1.0" ixy="0.0" ixz="0.0" iyy="1.0" iyz="0.0" izz="1.0" />
-      </inertial>
-      <visual>
-        <origin xyz="0 0 0" rpy="0 0 0" />
-        <geometry>
-          <box size="0.001 0.001 0.001" />
-        </geometry>
-      </visual>
-      <collision>
-        <origin xyz="0 0 ${-base_size_z / 2.0}" rpy="0 0 0" />
-        <geometry>
-          <box size="0.001 0.001 0.001" />
-        </geometry>
-      </collision>
-    </link>
-    <link name="${name}_link">
-      <inertial>
-        <mass value="${base_mass}" />
-        <origin xyz="0 0 0" />
-        <inertia ixx="5.652232699207" ixy="-0.009719934438" ixz="1.293988226423" iyy="5.669473158652" iyz="-0.007379583694" izz="3.683196351726" />
-      </inertial>
-      <visual>
-        <origin xyz="0 0 0" rpy="0 0 0" />
-        <geometry>
-          <mesh filename="package://youbot_description/meshes/youbot_base/base.dae"/>
-        </geometry>
-      </visual>
-    </link>
-    <front left wheel >
-    <link name="wheel_link_fl">
-      <inertial>
-        <mass value="${wheel_mass}" />
-        <origin xyz="0 0 0" />
-        <inertia  ixx="0.012411765597" ixy="-0.000711733678" ixz="0.00050272983" iyy="0.015218160428" iyz="-0.000004273467" izz="0.011763977943" />
-      </inertial>
-      <visual>
-        <origin xyz="0 0 0" rpy="0 0 0" />
-        <geometry>
-          <mesh filename="package://youbot_description/meshes/youbot_base/front-left_wheel.dae" />
-        </geometry>
-      </visual>
-      <collision>
-        <origin xyz="0 0 0" rpy="${M_PI/2} 0 0" />
-        <geometry>
-          <cylinder radius="${wheel_radius}" length="${wheel_radius}" />
-        </geometry>
-      </collision>
-    </link>
-    <front right wheel >
-    <link name="wheel_link_fr">
-      <inertial>
-        <mass value="${wheel_mass}" />
-        <origin xyz="0 0 0" />
-        <inertia  ixx="0.012411765597" ixy="-0.000711733678" ixz="0.00050272983" iyy="0.015218160428" iyz="-0.000004273467" izz="0.011763977943" />
-      </inertial>
-      <visual>
-        <origin xyz="0 0 0" rpy="0 0 0" />
-        <geometry>
-          <mesh filename="package://youbot_description/meshes/youbot_base/front-right_wheel.dae" />
-        </geometry>
-      </visual>
-      <collision>
-        <origin xyz="0 0 0" rpy="${M_PI/2} 0 0" />
-        <geometry>
-          <cylinder radius="${wheel_radius}" length="${wheel_radius}" />
-        </geometry>
-      </collision>
-    </link>
-    <back left wheel  >
-    <link name="wheel_link_bl">
-      <inertial>
-        <mass value="${wheel_mass}" />
-        <origin xyz="0 0 0" />
-        <inertia  ixx="0.012411765597" ixy="-0.000711733678" ixz="0.00050272983" iyy="0.015218160428" iyz="-0.000004273467" izz="0.011763977943" />
-      </inertial>
-      <visual>
-        <origin xyz="0 0 0" rpy="0 0 0" />
-        <geometry>
-          <mesh filename="package://youbot_description/meshes/youbot_base/back-left_wheel.dae" />
-        </geometry>
-      </visual>
-      <collision>
-        <origin xyz="0 0 0" rpy="${M_PI/2} 0 0" />
-        <geometry>
-          <cylinder radius="${wheel_radius}" length="${wheel_radius}" />
-        </geometry>
-      </collision>
-    </link>
-    < back right wheel  >
-    <link name="wheel_link_br">
-      <inertial>
-        <mass value="${wheel_mass}" />
-        <origin xyz="0 0 0" />
-        <inertia  ixx="0.012411765597" ixy="-0.000711733678" ixz="0.00050272983" iyy="0.015218160428" iyz="-0.000004273467" izz="0.011763977943" />
-      </inertial>
-      <visual>
-        <origin xyz="0 0 0" rpy="0 0 0" />
-        <geometry>
-          <mesh filename="package://youbot_description/meshes/youbot_base/back-right_wheel.dae" />
-        </geometry>
-      </visual>
-      <collision>
-        <origin xyz="0 0 0" rpy="${M_PI/2} 0 0" />
-        <geometry>
-          <cylinder radius="${wheel_radius}" length="${wheel_radius}" />
-        </geometry>
-      </collision>
-    </link>
-    < ### joints ### >
-    <joint name="${name}_footprint_joint" type="fixed">
-      <origin xyz="0 0 0" rpy="0 0 0" />
-      <child link="${name}_link" />
-      <parent link="${name}_footprint"/>
-    </joint>
-	-->
-    <!-- extensions -->

File: youbot_description/urdf/youbot_plate/plate.urdf.xacro (robot description, xacro)
@@ -1,32 +1,24 @@
 <?xml version="1.0"?>
+<!-- Refactored by Arn-O -->
 <robot name="youbot" xmlns:xacro="http://www.ros.org/wiki/xacro">
-	<xacro:include filename="$(find youbot_description)/urdf/youbot_plate/plate.gazebo.xacro" />
-	<xacro:macro name="youbot_plate" params="parent name *origin">
-		<!-- joint between arm_7_link and sdh_palm_link -->
-		<joint name="${name}_joint" type="fixed" >
-			<insert_block name="origin" />
-			<parent link="${parent}" />
-			<child link="${name}_link" />
-		</joint>
-		<link name="${name}_link">
-			<inertial>
-				<origin xyz="0 0 -0.025" rpy="0 0 0"/>
-				<mass value="1"/>
-				<inertia ixx="0.01" ixy="0" ixz="0" iyy="0.01" iyz="0" izz="0.01" />
-			</inertial>
-			<visual>
-				<origin xyz="0 0 -0.025" rpy="0 0 0" />
-				<geometry>
-					<mesh filename="package://youbot_description/meshes/youbot_plate/plate.dae" />
-				</geometry>
-			</visual>
-			<collision>
-				<origin xyz="0 0 -0.025" rpy="0 0 0" />
-				<geometry>
-					<mesh filename="package://youbot_description/meshes/youbot_plate/plate_convex.dae" />
-				</geometry>
-			</collision>
-		</link>
-		<xacro:youbot_plate_gazebo name="${name}" />
-	</xacro:macro>
+  <xacro:macro name="youbot_plate">
+  <!-- ### links ### -->
+  <link name="plate_link">
+    <inertial>
+     <mass value="${plate_mass}"/>
+     <inertia ixx="0.01" ixy="0" ixz="0" iyy="0.01" iyz="0" izz="0.01" />
+    </inertial>
+    <visual>
+      <geometry>
+        <mesh filename="package://youbot_description/meshes/youbot_plate/plate.dae" />
+      </geometry>
+    </visual>
+  </link>
+  <!-- ### joints ### -->
+  <joint name="$plate_joint" type="fixed" >
+    <origin xyz="${plate_pose_x} ${plate_pose_y} ${plate_pose_z}" rpy="0 0 0" />
+    <parent link="base_link" />
+    <child link="plate_link" />
+   </joint>
+  </xacro:macro>
 </robot>
