Commit message: nightly build

File: youbot_description/robots/youbot.urdf.xacro (robot description, xacro)
@@ -8,7 +8,10 @@
   <!-- youbot plate -->
   <xacro:include filename="$(find youbot_description)/urdf/youbot_plate/plate.urdf.xacro" />
+  <!-- youbot arm -->
+  <xacro:include filename="$(find youbot_description)/urdf/youbot_arm/arm.urdf.xacro" />
   <!-- generic simulator_gazebo plugins for starting mechanism control, ros time, ros battery -->
   <xacro:include filename="$(find youbot_description)/gazebo/gazebo.urdf.xacro" />
   <xacro:youbot_base />
   <xacro:youbot_plate />
+  <xacro:youbot_arm />
 </robot>

File: youbot_description/urdf/specs.urdf.xacro (robot description, xacro)
@@ -27,3 +27,8 @@
   <property name="plate_pose_y" value="0.000" />
   <property name="plate_pose_z" value="0.046" />
+  <!-- arm -->
+  <property name="arm_base_mass" value="0.961" />
+  <property name="arm_base_pose_x" value="0.143" />
+  <property name="arm_base_pose_y" value="0.000" />
+  <property name="arm_base_pose_z" value="0.046" />
 </robot>

File: youbot_description/urdf/youbot_arm/arm.urdf.xacro (robot description, xacro)
@@ -1,213 +1,29 @@
 <?xml version="1.0"?>
 <robot name="youbot" xmlns:xacro="http://www.ros.org/wiki/xacro">
-	<xacro:include filename="$(find youbot_description)/urdf/youbot_arm/arm.gazebo.xacro" />
-	<xacro:include filename="$(find youbot_description)/urdf/youbot_arm/arm.transmission.xacro" />
-	<xacro:include filename="$(find youbot_description)/urdf/youbot_arm/limits.urdf.xacro" />
-	<xacro:macro name="youbot_arm" params="parent name *origin">
-		<!-- joint between base_link and arm_0_link -->
-		<joint name="${name}_joint_0" type="fixed" >
-			<insert_block name="origin" />
-			<parent link="${parent}" />
-			<child link="${name}_link_0" />
-		</joint>
-		<link name="${name}_link_0">
-			<inertial>
-				<!--<origin xyz="0.023 0 0.006" rpy="0 0 0"/>-->
-				<origin xyz="0 0 0" rpy="0 0 0"/>
-				<mass value="${link_0_mass}"/>
-				<inertia ixx="0.01" ixy="0" ixz="0" iyy="0.01" iyz="0" izz="0.01" />
-			</inertial>
-			<visual>
-				<origin xyz="0 0 0" rpy="0 0 0" />
-				<geometry>
-					<mesh filename="package://youbot_description/meshes/youbot_arm/arm0.dae" />
-				</geometry>
-			</visual>
-			<collision>
-				<!--<origin xyz="0.023 0 0.006" rpy="0 0 0"/>-->
-				<origin xyz="0 0 0" rpy="0 0 0"/>
-				<geometry>
-					<mesh filename="package://youbot_description/meshes/youbot_arm/arm0_convex.dae" />
-					<!--<cylinder length="0.078" radius="0.093"/>-->
-				</geometry>
-			</collision>
-		</link>
-		<!-- joint between arm_0_link and arm_1_link -->
-		<joint name="${name}_joint_1" type="revolute">
-			<origin xyz="0.024 0 0.115" rpy="0 0 ${170 * M_PI / 180}"/>
-			<parent link="${name}_link_0"/>
-			<child link="${name}_link_1"/>
-			<axis xyz="0 0 -1"/>
-			<!--<calibration rising="${arm_1_ref}" falling="${arm_1_ref}"/>-->
-			<dynamics damping="1" friction="1" />
-			<!-- damping - N*s/m, N*s*m/rad -->
-			<!-- friction - N, N*m -->
-			<limit effort="${10000}" velocity="${M_PI / 2.0}" lower="0" upper="${joint_1_limit}"/>
-			<!--effort - N, N*m-->
-			<!--velocity - m/s, rad/s-->
-			<safety_controller k_position="20" k_velocity="${9.5/M_PI / 2.0}" soft_lower_limit="${threshold}" soft_upper_limit="${joint_1_limit_soft}" />
-			<!--k_position N/m, N/rad-->
-			<!--k_velocity N*s/m, N*s*m/rad-->
-			<!--for details: http://www.ros.org/wiki/pr2_controller_manager/safety_limits-->
-		</joint>
-		<link name="${name}_link_1">
-			<inertial>
-				<mass value="${link_1_mass}"/>
-				<xacro:link_1_inertia_tensor />
-			</inertial>
-			<visual>
-				<origin xyz="0 0 0" rpy="${M_PI} 0 0" />
-				<geometry>
-					<mesh filename="package://youbot_description/meshes/youbot_arm/arm1.dae" />
-				</geometry>
-			</visual>
-			<collision>
-				<!--<origin xyz="0 0 -0.003" rpy="0 0 0" />-->
-				<origin xyz="0 0 0" rpy="${M_PI} 0 0" />
-				<geometry>
-					<mesh filename="package://youbot_description/meshes/youbot_arm/arm_joint_1_convex.stl" />
-					<!--<cylinder length="0.102" radius="0.080"/>-->
-				</geometry>
-			</collision>
-		</link>
-		<!-- joint between arm_1_link and arm_2_link -->
-		<joint name="${name}_joint_2" type="revolute">
-			<origin xyz="0.033 0 0" rpy="0 ${-65 * M_PI / 180} 0"/>
-			<parent link="${name}_link_1"/>
-			<child link="${name}_link_2"/>
-			<axis xyz="0 1 0"/>
-			<!--<calibration rising="${arm_2_ref}" falling="${arm_2_ref}"/>-->
-			<dynamics damping="1" friction="1" />
-			<limit effort="${10000}" velocity="${M_PI / 2.0}" lower="0" upper="${joint_2_limit}"/>
-			<safety_controller k_position="20" k_velocity="${2*9.5/M_PI}" soft_lower_limit="${threshold}" soft_upper_limit="${joint_2_limit_soft}" />
-		</joint>
-		<link name="${name}_link_2">
-			<inertial>
-				<mass value="${link_2_mass}"/>
-				<xacro:link_2_inertia_tensor />
-			</inertial>
-			<visual>
-				<origin xyz="0 0 0" rpy="${- M_PI / 2} ${- M_PI / 2} 0" />
-				<geometry>
-					<mesh filename="package://youbot_description/meshes/youbot_arm/arm2.dae" />
-				</geometry>
-			</visual>
-			<collision>
-				<!--<origin xyz="0.001 -0.041 0.074" rpy="0 0 0" />-->
-				<origin xyz="0 0 0" rpy="${- M_PI / 2} ${- M_PI / 2} 0" />
-				<geometry>
-					<mesh filename="package://youbot_description/meshes/youbot_arm/arm_joint_2_convex.stl" />
-					<!--<box size="0.074 0.082 0.222"/>-->
-				</geometry>
-			</collision>
-		</link>
-		<joint name="${name}_joint_3" type="revolute">
-			<origin xyz="0.000 0.000 0.155" rpy="0 ${146 * M_PI / 180} 0"/>
-			<parent link="${name}_link_2"/>
-			<child link="${name}_link_3"/>
-			<axis xyz="0 1 0"/>
-			<dynamics damping="1" friction="1" />
-			<limit effort="${10000}" velocity="${M_PI / 2.0}" lower="-${joint_3_limit}" upper="0"/>
-			<safety_controller k_position="20" k_velocity="50" soft_lower_limit="-${joint_3_limit_soft}" soft_upper_limit="-${threshold}" />
-		</joint>
-		<link name="${name}_link_3">
-			<inertial>
-				<mass value="${link_3_mass}"/>
-				<xacro:link_3_inertia_tensor />
-			</inertial>
-			<visual>
-				<origin xyz="0 0 0" rpy="${M_PI / 2} 0 ${M_PI}" />
-				<geometry>
-					<mesh filename="package://youbot_description/meshes/youbot_arm/arm3.dae" />
-				</geometry>
-			</visual>
-			<collision>
-				<!--<origin xyz="0.000 0.025 0.067" rpy="0 0 0" />-->
-				<origin xyz="0 0 0" rpy="${M_PI / 2} 0 ${M_PI}" />
-				<geometry>
-					<mesh filename="package://youbot_description/meshes/youbot_arm/arm_joint_3_convex.stl" />
-					<!--<box size="0.064 0.054 0.192"/>-->
-				</geometry>
-			</collision>
-		</link>
-		<!-- joint between arm_3_link and arm_4_link -->
-		<joint name="${name}_joint_4" type="revolute">
-			<origin xyz="0.000 0.000 0.135" rpy="0 ${-102.5 * M_PI / 180} 0" />
-			<parent link="${name}_link_3"/>
-			<child link="${name}_link_4"/>
-			<axis xyz="0 1 0" />
-			<!--<calibration rising="${arm_4_ref}" falling="${arm_4_ref}"/>-->
-			<dynamics damping="1" friction="1" />
-			<limit effort="${10000}" velocity="${M_PI / 2.0}" lower="0" upper="${joint_4_limit}"/>
-			<safety_controller k_position="20" k_velocity="100" soft_lower_limit="0" soft_upper_limit="${joint_4_limit_soft}" />
-		</joint>
-		<link name="${name}_link_4">
-			<inertial>
-				<mass value="${link_4_mass}"/>
-				<xacro:link_4_inertia_tensor />
-			</inertial>
-			<visual>
-				<origin xyz="0 0 0" rpy="${M_PI / 2} 0 ${M_PI}"/>
-				<geometry>
-					<mesh filename="package://youbot_description/meshes/youbot_arm/arm4.dae" />
-				</geometry>
-			</visual>
-			<collision>
-				<!--<origin xyz="0 0 0.026" rpy="0 0 0" />-->
-				<origin xyz="0 0 0" rpy="${M_PI / 2} 0 ${M_PI}"/>
-				<geometry>
-					<mesh filename="package://youbot_description/meshes/youbot_arm/arm_joint_4_convex.stl" />
-					<!--<box size="0.058 0.100 0.118"/>-->
-				</geometry>
-			</collision>
-		</link>
-		<!-- joint between arm_4_link and arm_5_link -->
-		<joint name="${name}_joint_5" type="revolute">
-			<origin xyz="0 0 0.114" rpy="0 0 ${167.5 * M_PI / 180}" />
-			<parent link="${name}_link_4"/>
-			<child link="${name}_link_5"/>
-			<axis xyz="0 0 -1" />
-			<!--<calibration rising="${arm_5_ref}" falling="${arm_5_ref}"/>-->
-			<dynamics damping="1" friction="1" />
-			<limit effort="${10000}" velocity="${M_PI / 2.0}" lower="0" upper="${joint_5_limit}" />
-			<safety_controller k_position="20" k_velocity="100" soft_lower_limit="0" soft_upper_limit="${joint_5_limit_soft}" />
-		</joint>
-		<link name="${name}_link_5">
-			<inertial>
-				<mass value="${link_5_mass}"/>
-				<xacro:link_5_inertia_tensor />
-			</inertial>
-			<visual>
-				<origin xyz="0 0 0" rpy="0 0 0" />
-				<geometry>
-					<mesh filename="package://youbot_description/meshes/youbot_arm/arm5.dae" />
-				</geometry>
-			</visual>
-			<collision>
-				<origin xyz="0 0 0" rpy="0 0 0" />
-				<geometry>
-					<mesh filename="package://youbot_description/meshes/youbot_arm/arm_joint_5_convex.stl" />
-					<!--<box size="0.054 0.096 0.030"/>-->
-				</geometry>
-			</collision>
-		</link>
-<!--
-    <joint name="${name}_joint_6_dummy" type="revolute">
-      <origin xyz="0 0 0" rpy="0 0 0"/>
-      <parent link="${name}_link_5"/>
-      <child link="${name}_link_6_dummy"/>
-      <axis xyz="0 0 1"/>
-      <limit effort="1" velocity="${M_PI / 2.0}" lower="0" upper="${2 * M_PI}" />
+  <!-- xacro:include filename="$(find youbot_description)/urdf/youbot_arm/arm.transmission.xacro" /-->
+  <!-- uncomment for adding the controllers -->
+  <xacro:include filename="$(find youbot_description)/urdf/specs.urdf.xacro" />
+  <xacro:macro name="youbot_arm">
+    <!-- ### links ### -->
+    <link name="arm_base_link">
+      <inertial>
+        <mass value="${arm_base_mass}" />
+        <inertia ixx="0.010" ixy="0.000" ixz="0.000" iyy="0.010" iyz="0.000" izz="0.010" />
+      </inertial>
+      <visual>
+        <geometry>
+          <mesh filename="package://youbot_description/meshes/youbot_arm/arm_base_frame.dae"/>
+        </geometry>
+      </visual>
+    </link>
+    <!-- ### joints ### -->
+    <joint name="arm_base_joint" type="fixed">
+      <origin xyz="${arm_base_pose_x} ${arm_base_pose_y} ${arm_base_pose_z}" rpy="0 0 0" />
+      <parent link="base_link"/>
+      <child link="arm_base_link" />
     </joint>
-		<link name="${name}_link_6_dummy">
-			<inertial>
-				<mass value="0.001"/>
-				<xacro:link_5_inertia_tensor />
-			</inertial>
-		</link>
-	-->
-	<!-- extensions -->
-	<xacro:youbot_arm_gazebo name="${name}" />
-	<xacro:youbot_arm_transmission name="${name}" />
-</xacro:macro>
+    <!-- extensions -->
+    <!-- uncomment for adding the controllers -->
+    <!-- xacro:youbot_arm_transmission /-->
+  </xacro:macro>
 </robot>

File: youbot_description/urdf/youbot_base/base.gazebo.xacro (robot description, xacro)
@@ -1,4 +1,5 @@
 <?xml version="1.0"?>
 <!-- Refactored by Arn-O -->
+<!-- TODO should be moved to gazebo general file? -->
 <robot name="youbot" xmlns:xacro="http://www.ros.org/wiki/xacro">
   <xacro:macro name="youbot_base_gazebo">

File: youbot_description/urdf/youbot_base/base.urdf.xacro (robot description, xacro)
@@ -4,5 +4,5 @@
   <!-- includes -->
   <xacro:include filename="$(find youbot_description)/urdf/specs.urdf.xacro" />
-  <xacro:include filename="$(find youbot_description)/urdf/youbot_base/base.gazebo.xacro" />
+  <!-- xacro:include filename="$(find youbot_description)/urdf/youbot_base/base.gazebo.xacro" /-->
   <xacro:macro name="youbot_base">
     <!-- ### links ### -->
