Commit message: nightly build

File: youbot_description/urdf/specs.urdf.xacro (robot description, xacro)
@@ -32,3 +32,10 @@
   <property name="arm_base_pose_y" value="0.000" />
   <property name="arm_base_pose_z" value="0.046" />
+  <property name="arm_1_link_mass" value="1.390" />
+  <property name="arm_1_link_pose_x" value="0.024" />
+  <property name="arm_1_link_pose_y" value="0.000" />
+  <property name="arm_1_link_pose_z" value="0.115" />
+  <property name="arm_1_link_orient_z" value="${M_PI * (0 / 180)}" />
+  <property name="arm_1_link_orient_y" value="${M_PI * (0 / 180)}" />
+  <property name="arm_1_link_orient_x" value="${M_PI * (180 / 180)}" />
 </robot>

File: youbot_description/urdf/youbot_arm/arm.urdf.xacro (robot description, xacro)
@@ -17,4 +17,15 @@
       </visual>
     </link>
+    <link name="arm_1_link">
+      <inertial>
+        <mass value="${arm_1_link_mass}" />
+        <inertia ixx="0.010" ixy="0.000" ixz="0.000" iyy="0.010" iyz="0.000" izz="0.010" />
+      </inertial>
+      <visual>
+        <geometry>
+          <mesh filename="package://youbot_description/meshes/youbot_arm/arm_joint_1.dae"/>
+        </geometry>
+      </visual>
+    </link>
     <!-- ### joints ### -->
     <joint name="arm_base_joint" type="fixed">
@@ -23,4 +34,10 @@
       <child link="arm_base_link" />
     </joint>
+    <joint name="arm_1_joint" type="fixed">
+      <origin xyz="${arm_1_link_pose_x} ${arm_1_link_pose_y} ${arm_1_link_pose_z}"
+              rpy="${arm_1_link_orient_x} ${arm_1_link_orient_y} ${arm_1_link_orient_z}" />
+      <parent link="arm_base_link"/>
+      <child link="arm_1_link" />
+    </joint>
     <!-- extensions -->
     <!-- uncomment for adding the controllers -->

Commit message: nightly built

File: youbot_description/urdf/specs.urdf.xacro (robot description, xacro)
@@ -39,3 +39,10 @@
   <property name="arm_1_link_orient_y" value="${M_PI * (0 / 180)}" />
   <property name="arm_1_link_orient_x" value="${M_PI * (180 / 180)}" />
+  <property name="arm_2_link_mass" value="1.318" />
+  <property name="arm_2_link_pose_x" value="0.033" />
+  <property name="arm_2_link_pose_y" value="0.000" />
+  <property name="arm_2_link_pose_z" value="0.000" />
+  <property name="arm_2_link_orient_z" value="${M_PI * (0 / 180)}" />
+  <property name="arm_2_link_orient_y" value="${M_PI * (0 / 180)}" />
+  <property name="arm_2_link_orient_x" value="${M_PI * (0 / 180)}" />
 </robot>

File: youbot_description/urdf/youbot_arm/arm.urdf.xacro (robot description, xacro)
@@ -28,4 +28,15 @@
       </visual>
     </link>
+    <link name="arm_2_link">
+      <inertial>
+        <mass value="${arm_2_link_mass}" />
+        <inertia ixx="0.010" ixy="0.000" ixz="0.000" iyy="0.010" iyz="0.000" izz="0.010" />
+      </inertial>
+      <visual>
+        <geometry>
+          <mesh filename="package://youbot_description/meshes/youbot_arm/arm_joint_2.dae"/>
+        </geometry>
+      </visual>
+    </link>
     <!-- ### joints ### -->
     <joint name="arm_base_joint" type="fixed">
@@ -40,4 +51,10 @@
       <child link="arm_1_link" />
     </joint>
+    <joint name="arm_2_joint" type="fixed">
+      <origin xyz="${arm_2_link_pose_x} ${arm_2_link_pose_y} ${arm_2_link_pose_z}"
+              rpy="${arm_2_link_orient_x} ${arm_2_link_orient_y} ${arm_2_link_orient_z}" />
+      <parent link="arm_1_link"/>
+      <child link="arm_2_link" />
+    </joint>
     <!-- extensions -->
     <!-- uncomment for adding the controllers -->

Commit message: nightly build

File: youbot_description/urdf/specs.urdf.xacro (robot description, xacro)
@@ -36,13 +36,13 @@
   <property name="arm_1_link_pose_y" value="0.000" />
   <property name="arm_1_link_pose_z" value="0.115" />
-  <property name="arm_1_link_orient_z" value="${M_PI * (0 / 180)}" />
   <property name="arm_1_link_orient_y" value="${M_PI * (0 / 180)}" />
-  <property name="arm_1_link_orient_x" value="${M_PI * (180 / 180)}" />
+  <property name="arm_1_link_orient_p" value="${M_PI * (0 / 180)}" />
+  <property name="arm_1_link_orient_r" value="${M_PI * (180 / 180)}" />
   <property name="arm_2_link_mass" value="1.318" />
   <property name="arm_2_link_pose_x" value="0.033" />
   <property name="arm_2_link_pose_y" value="0.000" />
   <property name="arm_2_link_pose_z" value="0.000" />
-  <property name="arm_2_link_orient_z" value="${M_PI * (0 / 180)}" />
-  <property name="arm_2_link_orient_y" value="${M_PI * (0 / 180)}" />
-  <property name="arm_2_link_orient_x" value="${M_PI * (0 / 180)}" />
+  <property name="arm_2_link_orient_y" value="${M_PI * (-90 / 180)}" />
+  <property name="arm_2_link_orient_p" value="${M_PI * (0 / 180)}" />
+  <property name="arm_2_link_orient_r" value="${M_PI * (90 / 180)}" />
 </robot>

File: youbot_description/urdf/youbot_arm/arm.urdf.xacro (robot description, xacro)
@@ -45,15 +45,17 @@
       <child link="arm_base_link" />
     </joint>
-    <joint name="arm_1_joint" type="fixed">
+    <joint name="arm_1_joint" type="revolute">
       <origin xyz="${arm_1_link_pose_x} ${arm_1_link_pose_y} ${arm_1_link_pose_z}"
-              rpy="${arm_1_link_orient_x} ${arm_1_link_orient_y} ${arm_1_link_orient_z}" />
+              rpy="${arm_1_link_orient_r} ${arm_1_link_orient_p} ${arm_1_link_orient_y}" />
       <parent link="arm_base_link"/>
       <child link="arm_1_link" />
+      <limit lower="-2.0" upper="2.0" effort="1000" velocity="3" />
     </joint>
-    <joint name="arm_2_joint" type="fixed">
+    <joint name="arm_2_joint" type="revolute">
       <origin xyz="${arm_2_link_pose_x} ${arm_2_link_pose_y} ${arm_2_link_pose_z}"
-              rpy="${arm_2_link_orient_x} ${arm_2_link_orient_y} ${arm_2_link_orient_z}" />
+              rpy="${arm_2_link_orient_r} ${arm_2_link_orient_p} ${arm_2_link_orient_y}" />
       <parent link="arm_1_link"/>
       <child link="arm_2_link" />
+      <limit lower="-2.0" upper="2.0" effort="1000" velocity="3" />
     </joint>
     <!-- extensions -->
