Commit message: Solved minor issues

File: youbot_description/urdf/sensors/hokuyo_urg04_laser.gazebo.xacro (robot description, xacro)
@@ -7,4 +7,5 @@
         <gazebo reference="${name}_link">
             <sensor name="${name}" type="ray">
+                <visualize>true</visualize>
                 <ray>
                     <scan>
@@ -12,6 +13,6 @@
                             <samples>640</samples>
                             <resolution>1.0</resolution>
-                            <min_angle>${min_angle*180.0/M_PI}</min_angle>
-                            <max_angle>${max_angle*180.0/M_PI}</max_angle>
+                            <min_angle>${min_angle}</min_angle>
+                            <max_angle>${max_angle}</max_angle>
                         </horizontal>
                     </scan>
@@ -27,5 +28,5 @@
                     <updateRate>${update_rate}</updateRate>
                     <topicName>${ros_topic}</topicName>
-                    <frameName>/${name}_link</frameName>
+                    <frameName>${name}_link</frameName>
                     <interface:laser name="gazebo_ros_${name}_iface" />
                 </plugin>

File: youbot_description/urdf/sensors/hokuyo_urg04_laser.urdf.xacro (robot description, xacro)
@@ -17,18 +17,18 @@
       <visual>
       	<origin xyz="0 0 0" rpy="0 0 0" />
-	<geometry>
-		<mesh filename="package://youbot_description/meshes/sensors/hokuyo.dae" />
-	</geometry>
-	<material name="DarkGrey" />
-      </visual>
-      <collision>
-		<origin xyz="0 0 0" rpy="0 0 0" />
-		<geometry>
-			<mesh filename="package://youbot_description/meshes/sensors/hokuyo_convex.dae" />
-		</geometry>
-	</collision>
-    </link>
-    <!-- gazebo extensions -->
-    <xacro:hokuyo_urg04_laser_gazebo name="${name}" ros_topic="${ros_topic}" update_rate="${update_rate}" min_angle="${min_angle}" max_angle="${max_angle}" />
-  </xacro:macro>
+       <geometry>
+        <mesh filename="package://youbot_description/meshes/sensors/hokuyo.dae" />
+      </geometry>
+      <material name="DarkGrey" />
+    </visual>
+    <collision>
+      <origin xyz="0 0 0" rpy="0 0 0" />
+      <geometry>
+       <mesh filename="package://youbot_description/meshes/sensors/hokuyo_convex.dae" />
+     </geometry>
+   </collision>
+ </link>
+ <!-- gazebo extensions -->
+ <xacro:hokuyo_urg04_laser_gazebo name="${name}" ros_topic="${ros_topic}" update_rate="${update_rate}" min_angle="${min_angle}" max_angle="${max_angle}" />
+</xacro:macro>
 </robot>

File: youbot_description/urdf/youbot_base/base.gazebo.xacro (robot description, xacro)
@@ -8,5 +8,5 @@
         <odometryFrame>odom</odometryFrame>
         <odometryRate>20.0</odometryRate>
-        <robotBaseFrame>base_footprint</robotBaseFrame>
+        <robotBaseFrame>base_link</robotBaseFrame>
       </plugin>
     </gazebo>
@@ -15,20 +15,4 @@
       <selfCollide>true</selfCollide>
     </gazebo>
-    <!-- old position controller -->
-    <!--
-      <plugin name="p3d_base_controller" filename="libgazebo_ros_p3d.so">
-        <alwaysOn>true</alwaysOn>
-        <updateRate>100.0</updateRate>
-        <bodyName>base_link</bodyName>
-        <topicName>base_pose_ground_truth</topicName>
-        <gaussianNoise>0.01</gaussianNoise>
-        <frameName>map</frameName>
-        <xyzOffsets>25.7 25.7 0</xyzOffsets>  initialize odometry for fake localization
-        <rpyOffsets>0 0 0</rpyOffsets>
-        <interface:position name="p3d_base_position"/>
-      </plugin>
-      <canonicalBody>base_footprint</canonicalBody>
-    </gazebo>
-  -->
 </xacro:macro>
 </robot>

File: youbot_description/urdf/youbot_base/base.urdf.xacro (robot description, xacro)
@@ -246,5 +246,5 @@
     <!-- base laser front -->
     <xacro:hokuyo_urg04_laser name="${name}_laser_front" parent="${name}" ros_topic="scan_front" update_rate="10" min_angle="-1.57" max_angle="1.57" >
-      <origin xyz="0.3 0 -0.03" rpy="3.15 3.15 0" />
+      <origin xyz="0.3 0 -0.03" rpy="${M_PI} ${M_PI} ${M_PI}" />
     </xacro:hokuyo_urg04_laser>
     <!-- extensions -->
